File: Console-Controller/LTC4412HV.sch (KiCad schematic (older format))
At the start: 5 parts, among them Q3 Si7463DP, U9 LTC4412HVIS6

Commit message: latest WIP, LTC1760 module ready for layout, strone-controller ready for layout but needs mech board drawings
Parts:
- removed C26, C27: 0.1 uF 50V, Capacitor_SMD:C_0603_1608Metric_Pad1.05x0.95mm_HandSolder, symbol Device:C_Small
- removed Q3: Si7463DP, Package_SO:PowerPAK_SO-8_Single, symbol ProjectDevices:Si7463DP
- removed R26: 470k, Resistor_SMD:R_0603_1608Metric_Pad1.05x0.95mm_HandSolder, symbol Device:R_Small_US
- removed U9: LTC4412HVIS6, Package_TO_SOT_SMD:TSOT-23-6, symbol Power_Management:LTC4412xS6
- added C1, C2: 0.1 uF 50V, Capacitor_SMD:C_0603_1608Metric_Pad1.05x0.95mm_HandSolder, symbol Device:C_Small
- added Q1: Si7463DP, Package_SO:PowerPAK_SO-8_Single, symbol Dual-Mag-Camera-Control-rescue:Si7463DP-ProjectDevices
- added R8: 470k, Resistor_SMD:R_0603_1608Metric_Pad1.05x0.95mm_HandSolder, symbol Device:R_Small_US
- added TP1: STAT, symbol Connector:TestPoint
- added U13: LTC4412HVIS6, Package_TO_SOT_SMD:TSOT-23-6, symbol Power_Management:LTC4412xS6
