File: Console-Controller/COMMS.kicad_sch (KiCad schematic)
At the start: 44 parts, among them J10 RS-232_2_3, J7 UART_0_1, J8 UART_2_3, J9 RS-232_0_1

Commit message: slight updates to LTC1670 modules (2 resistors added) finalizing console controller and strobe controller
Parts:
- removed D25, D26, D27, D28, D29, D30, D31, D32: CZRU52C3V3, Diode_SMD:D_0603_1608Metric_Pad1.05x0.95mm_HandSolder, symbol 2022-05-02_03-27-09:CZRU52C3V3
- removed D? (x8): TESDU12V RGG, Resistor_SMD:R_0603_1608Metric, symbol Diode:SD36_SOD323
- removed F15, F16, F17, F18, F19, F20, F21, F22, F23, F24, F25, F26, F27, F28, F29, F30: PTC, Resistor_SMD:R_1210_3225Metric_Pad1.42x2.65mm_HandSolder, symbol Dual-Mag-Camera-Control-rescue:Polyfuse_Small-SPC-Control-rescue
- removed J10: RS-232_2_3, Connector_Molex:Molex_Nano-Fit_105310-xx06_2x03_P2.50mm_Vertical, symbol Dual-Mag-Camera-Control-rescue:Conn_01x06-SPC-Control-rescue
- removed J7: UART_0_1, Connector_Molex:Molex_Nano-Fit_105310-xx06_2x03_P2.50mm_Vertical, symbol Dual-Mag-Camera-Control-rescue:Conn_01x06-SPC-Control-rescue
- removed J8: UART_2_3, Connector_Molex:Molex_Nano-Fit_105310-xx06_2x03_P2.50mm_Vertical, symbol Dual-Mag-Camera-Control-rescue:Conn_01x06-SPC-Control-rescue
- removed J9: RS-232_0_1, Connector_Molex:Molex_Nano-Fit_105310-xx06_2x03_P2.50mm_Vertical, symbol Dual-Mag-Camera-Control-rescue:Conn_01x06-SPC-Control-rescue
- removed JP10, JP11, JP12, JP13, JP14, JP15, JP8, JP9: (no value), Jumper:SolderJumper-2_P1.3mm_Open_RoundedPad1.0x1.5mm, symbol Jumper:SolderJumper_2_Open
- added C14, C15, C16, C17, C18, C19, C? (x6): 100 nF, Capacitor_SMD:C_0603_1608Metric, symbol EyeRIS-LRAUV-Control-rescue:C_Small-SPC-Control-rescue-EyeRIS-LRAUV-Control-res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
- added D34, D82, D? (x6): CDSOD323-T15C, Diode_SMD:D_SOD-323, symbol Dual-Mag-Camera-Control-rescue:D_TVS-SPC-Control-rescue
- added D? (x8): CDSOD323-T03C, Diode_SMD:D_SOD-323, symbol Dual-Mag-Camera-Control-rescue:D_TVS-SPC-Control-rescue
- added F1, F2, F? (x14): PTC, Resistor_SMD:R_1210_3225Metric, symbol Dual-Mag-Camera-Control-rescue:Polyfuse_Small-SPC-Control-rescue
- added J9, J?: RS-232 0, Connector_Molex:Molex_PicoBlade_53261-0371_1x03-1MP_P1.25mm_Horizontal, symbol Connector_Generic:Conn_01x03
- added J? (x2): RS-232 1, Connector_Molex:Molex_PicoBlade_53261-0371_1x03-1MP_P1.25mm_Horizontal, symbol Connector_Generic:Conn_01x03
- added J?: UART 0, Connector_Molex:Molex_PicoBlade_53261-0371_1x03-1MP_P1.25mm_Horizontal, symbol Connector_Generic:Conn_01x03
- added J?: UART PASS 0, Connector_Molex:Molex_PicoBlade_53261-0371_1x03-1MP_P1.25mm_Horizontal, symbol Connector_Generic:Conn_01x03
- added J?: UART 1, Connector_Molex:Molex_PicoBlade_53261-0371_1x03-1MP_P1.25mm_Horizontal, symbol Connector_Generic:Conn_01x03
- added J?: UART PASS 1, Connector_Molex:Molex_PicoBlade_53261-0371_1x03-1MP_P1.25mm_Horizontal, symbol Connector_Generic:Conn_01x03
- added U10: MAX3232E, Package_SO:TSSOP-16_4.4x5mm_P0.65mm, symbol EyeRIS-LRAUV-Control-rescue:MAX3232E-SPC-Control-rescue-EyeRIS-LRAUV-Control-re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
- added U?: MAX3232E-QE, Package_SO:TSSOP-16_4.4x5mm_P0.65mm, symbol EyeRIS-LRAUV-Control-rescue:MAX3232E-SPC-Control-rescue-EyeRIS-LRAUV-Control-re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
Connections:
- net PGND: now also C16.2, C17.2, C18.2, C19.1, C?.1, C?.2, C?.2, C?.2, D34.2 (A2), D82.2 (A2), D?.2 (A2), D?.2 (A2), D?.2 (A2), D?.2 (A2), D?.2 (A2), D?.2 (A2), D?.2 (A2), D?.2 (A2), D?.2 (A2), D?.2 (A2), D?.2 (A2), D?.2 (A2), D?.2 (A2), D?.2 (A2), J9.3 (Pin_3), J?.3 (Pin_3), J?.3 (Pin_3), J?.3 (Pin_3), J?.3 (Pin_3), J?.3 (Pin_3), J?.3 (Pin_3), J?.3 (Pin_3), U10.15 (GND), U?.15 (GND)
- net UART_RX0: now also U10.12 (R1OUT)
- net UART_RX1: now also U10.9 (R2OUT)
- net UART_RX2: now also D?.1 (A1), F?.2
- net UART_RX3: now also D?.1 (A1), F?.2
- net UART_TX0: now also U10.11 (T1IN)
- net UART_TX1: now also U10.10 (T2IN)
- net UART_TX2: now also D?.1 (A1), F?.2
- net UART_TX3: now also D?.1 (A1), F?.2
- new net: F?.1, J?.1 (Pin_1) (x7)
- new net: D?.1 (A1), F?.2, U10.7 (T2OUT)
- new net: F1.1, J9.1 (Pin_1)
- new net: D34.1 (A1), F1.2, U10.14 (T1OUT)
- new net: D?.1 (A1), F?.2, U?.10 (T2IN)
- new net: C14.2, U10.1 (C1+)
- new net: D82.1 (A1), F2.2, U10.13 (R1IN)
- new net: C18.1, U10.2 (V+)
- new net: C14.1, U10.3 (C1-)
- new net: C15.2, U10.4 (C2+)
- new net: C15.1, U10.5 (C2-)
- new net: C19.2, U10.6 (V-)
- new net: D?.1 (A1), F?.2, U10.8 (R2IN)
- new net: F?.1, J?.2 (Pin_2) (x7)
- new net: D?.1 (A1), F?.2, U?.14 (T1OUT)
- new net: C?.1, U?.5 (C2-)
- new net: C?.2, U?.4 (C2+)
- new net: D?.1 (A1), F?.2, U?.11 (T1IN)
- new net: C?.1, U?.3 (C1-)
- new net: C?.2, U?.1 (C1+)
- new net: D?.1 (A1), F?.2, U?.7 (T2OUT)
- new net: D?.1 (A1), F?.2, U?.12 (R1OUT)
- new net: F2.1, J9.2 (Pin_2)
- new net: C?.2, U?.6 (V-)
- new net: C?.1, U?.2 (V+)
- new net: D?.1 (A1), F?.2, U?.13 (R1IN)
- new net: D?.1 (A1), F?.2, U?.8 (R2IN)
- new net: D?.1 (A1), F?.2, U?.9 (R2OUT)
- new net 3V3: C16.1, C17.1, C?.1, C?.1, U10.16 (VCC), U?.16 (VCC)
Other:
- removed sheet Sparkfun_MAX3232
- removed sheet Sparkfun_MAX3233
- note added: "SAMD21 UART I/O Protection fuses and dioes on UART Lines"
- note added: "SAMD21 UART to RS-232 I/O Protection fuses and dioes on RS-232"
- note added: "UART to RS-232 Converter Pass through either direction without going through SAMD21 controller"
