File: Console-Controller/Console-Controller.kicad_sch (KiCad schematic)
At the start: 9 parts, among them J1 Charge Input, J2 Battery Output, J21 BATT_EN, Q10 SiSA72DN

Commit message: latest WIP, LTC1760 module ready for layout, strone-controller ready for layout but needs mech board drawings
Parts:
- removed D11: BZT52C20T-7, Diode_SMD:D_SOD-523, symbol BUMP-Control-rescue:ZENERsmall-RESCUE-PowerControlBoard-SPC-Control-rescue-Deat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
- removed F1: 10 A, ProjectFootprints:01550900M, symbol WW-Battery-Pack-rescue:small_fuse-ProjectDevices
- removed F? (x2): 3A 36V, ProjectFootprints:MF-GSMF, symbol Device:Polyfuse_Small
- removed J1: Charge Input, Connector_Molex:Molex_Mini-Fit_Jr_5566-04A_2x02_P4.20mm_Vertical, symbol Connector_Generic:Conn_01x04
- removed J2: Battery Output, Connector_Molex:Molex_Mini-Fit_Jr_5566-06A_2x03_P4.20mm_Vertical, symbol Connector_Generic:Conn_01x06
- removed J21: BATT_EN, Connector_PinHeader_2.54mm:PinHeader_1x02_P2.54mm_Vertical, symbol Connector_Generic:Conn_01x02
- removed Q10: SiSA72DN, ProjectFootprints:PowerPAK 1212, symbol ProjectDevices:SiSA72DN
- removed R79: 10K, Resistor_SMD:R_0603_1608Metric_Pad1.05x0.95mm_HandSolder, symbol BUMP-Control-rescue:Resistor_small-SPC-Control-rescue-DeathStar-rescue
- added D1: GRN 1.7V@1mA, LED_SMD:LED_0603_1608Metric, symbol Device:LED_Small_ALT
- added D10, D11, D12, D13, D14, D15, D16, D4, D5, D6, D7, D8, D9: CZRU52C3V3, Diode_SMD:D_0603_1608Metric_Pad1.05x0.95mm_HandSolder, symbol 2022-05-02_03-27-09:CZRU52C3V3
- added D2, D3: ORG 1.8V@1mA, LED_SMD:LED_0603_1608Metric, symbol Device:LED_Small_ALT
- added F10, F11, F12, F13, F14, F2, F3, F4, F5, F6, F7, F8, F9: PTC, Resistor_SMD:R_1210_3225Metric, symbol Dual-Mag-Camera-Control-rescue:Polyfuse_Small-SPC-Control-rescue
- added J1: ~TRIG_IO, Connector_Molex:Molex_Nano-Fit_105310-xx06_2x03_P2.50mm_Vertical, symbol Dual-Mag-Camera-Control-rescue:Conn_01x06-SPC-Control-rescue
- added J13: STRB_PWR, Connector_Molex:Molex_Nano-Fit_105309-xx02_1x02_P2.50mm_Vertical, symbol Connector_Generic:Conn_01x02
- added J14: CAM_COMPUTE_PWR, Connector_Molex:Molex_Nano-Fit_105309-xx02_1x02_P2.50mm_Vertical, symbol Connector_Generic:Conn_01x02
- added J15: 5V_5A_PWR, Connector_Molex:Molex_Nano-Fit_105309-xx02_1x02_P2.50mm_Vertical, symbol Connector_Generic:Conn_01x02
- added J16: 5V_2.5A_PWR, Connector_Molex:Molex_Nano-Fit_105309-xx02_1x02_P2.50mm_Vertical, symbol Connector_Generic:Conn_01x02
- added J2: TRIG_IO, Connector_Molex:Molex_Nano-Fit_105310-xx06_2x03_P2.50mm_Vertical, symbol Dual-Mag-Camera-Control-rescue:Conn_01x06-SPC-Control-rescue
- added J3: ADC_DAC, Connector_Molex:Molex_Nano-Fit_105310-xx06_2x03_P2.50mm_Vertical, symbol Dual-Mag-Camera-Control-rescue:Conn_01x06-SPC-Control-rescue
- added J4: GPIO, Connector_Molex:Molex_Nano-Fit_105310-xx06_2x03_P2.50mm_Vertical, symbol Dual-Mag-Camera-Control-rescue:Conn_01x06-SPC-Control-rescue
- added R1, R2, R3: 3240, Resistor_SMD:R_0603_1608Metric_Pad1.05x0.95mm_HandSolder, symbol Device:R_Small_US
- added R19, R20: 10K, Resistor_SMD:R_0603_1608Metric_Pad1.05x0.95mm_HandSolder, symbol Dual-Mag-Camera-Control-rescue:Resistor_small-SPC-Control-rescue-DeathStar-resc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
- added R4, R5, R6: 1k, Resistor_SMD:R_0603_1608Metric_Pad1.05x0.95mm_HandSolder, symbol Device:R_Small_US
- added U1: D24V10F5, ProjectFootprints:D24V10F5, symbol Dual-Mag-Camera-Control-rescue:D24V10F5-ProjectDevices
- added U3: D24V50F5, ProjectFootprints:D24V50F5, symbol Dual-Mag-Camera-Control-rescue:D24V50F5-ProjectDevices
- added U4: LowPowerLab-SD-Card, ProjectFootprints:LowPowerLabs-SD-Card, symbol Dual-Mag-Camera-Control-rescue:LowPowerLab-SD-Card-ProjectDevices
- added U5: D24V22F5, ProjectFootprints:D24V22F5, symbol Dual-Mag-Camera-Control-rescue:D24V22F5-ProjectDevices
- added U8: MoteinoM0, ProjectFootprints:MoteinoM0, symbol Dual-Mag-Camera-Control-rescue:MoteinoM0-ProjectDevices
Connections:
- net GND: now also D1.1 (K), D10.2, D11.2, D12.2, D13.2, D14.2, D15.2, D16.2, D2.1 (K), D3.1 (K), D4.2, D5.2, D6.2, D7.2, D8.2, D9.2, J1.6 (Pin_6), J13.2 (Pin_2), J14.2 (Pin_2), J15.2 (Pin_2), J16.2 (Pin_2), J2.6 (Pin_6), J3.6 (Pin_6), J4.6 (Pin_6), U1.4 (GND), U3.2 (GND), U3.3 (GND), U4.1 (GND), U4.14 (GND), U5.2 (GND), U8.2 (GND), U8.31 (GND), U8.33 (GND)
- new net: D1.2 (A), R1.2, U1.1 (PG)
- new net: D3.2 (A), R3.1
- new net: D2.2 (A), R2.1
- new net 3.3V_LDO: J1.4 (Pin_4), J2.4 (Pin_4), J3.5 (Pin_5), J4.4 (Pin_4), R19.1, R20.1, R4.2, R5.2, R6.2, U4.2 (3V), U8.30 (3.3V_LDO), U8.34 (3.3V_LDO)
- new net 5V_2.5A_OUT: J16.1 (Pin_1), R3.2, U5.1 (Vout)
- new net 5V_5A_OUT: J15.1 (Pin_1), R2.2, U3.1 (Out)
- new net 5V_reg: J1.5 (Pin_5), J2.5 (Pin_5), J4.5 (Pin_5), R1.1, U1.5 (Vout), U8.32 (Vin_(3.6V-6V))
- new net A3: D6.1, F4.1, U8.11 (A3(PA04(AIN4/REFB/SER0:0/TC0:0)))
- new net A3_IO: F4.2, J3.1 (Pin_1)
- new net A4: D11.1, F9.1, U8.10 (A4(PA05(AIN5/SER0:1/TC0:1)))
- new net A4_IO: F9.2, J3.2 (Pin_2)
- new net A5: D15.1, F13.1, U8.9 (A5(PB02(AIN10/SER5:0))
- new net A5_IO: F13.2, J3.3 (Pin_3)
- new net CamVout: J14.1 (Pin_1)
- new net DAC_OUT: D8.1, F6.1, U8.14 (A0(PA02(AIN0/DAC)))
- new net DAC_OUT_IO: F6.2, J3.4 (Pin_4)
- new net GPIO_1: D7.1, F5.1, U4.12 (CD), U8.37 (AREF(PA03(AIN1/REFA)))
- new net GPIO_1_IO: F5.2, J4.1 (Pin_1)
- new net GPIO_2: D12.1, F10.1, U8.36 (SWDIO(PA31(SWDIO/SER1:3+)))
- new net GPIO_2_IO: F10.2, J4.2 (Pin_2)
- new net GPIO_3: D16.1, F14.1, U8.35 (SWCLK(PA30(SWCLK/SER1:2+)))
- new net GPIO_3_IO: F14.2, J4.3 (Pin_3)
- new net SCL_1: R19.2, U8.29 (SCL(PA23(I2C/SER3:0+)))
- new net SDA_1: R20.2, U8.28 (SDA(PA22(I2C/SER3:0+)))
- new net SD_CS: U4.10 (CS), U8.3 (D13(PA17(I2C/SER1:1+)))
- new net SD_ENABLE: U4.11 (EN), U8.5 (D11(PA16(I2C/SER1:0+)))
- new net SPI_MISO: U4.5 (MI), U8.27 (SPI_MISO(PA12(I2C/SER2:0+)))
- new net SPI_MOSI: U4.7 (MO), U8.25 (SPI_MOSI(PB10(SER4:2+)))
- new net SPI_SCK: U4.6 (SCK), U8.26 (SPI_SCK(PB11(SER4:3+)))
- new net Serial0_RX: U8.8 (D31(PB23(SER5:3+)))
- new net Serial0_TX: U8.7 (D30(PB22(SER5:2+)))
- new net Serial1_RX: U8.24 (D0(PA11(AIN19/SER0:3+)))
- new net Serial1_TX: U8.23 (D1(PA10(AIN18/SER0:2+)))
- new net Serial2_RX: U8.19 (D5(PA15(XOUT/SER2:3+)))
- new net Serial2_TX: U8.22 (D2(PA14(XIN/SER2:2+)))
- new net Serial3_RX: U8.4 (D12(PA19(SER1:3+)))
- new net Serial3_TX: U8.6 (D10(PA18(SER1:2+)))
- new net StrobeVout: J13.1 (Pin_1)
- new net SystemVin: U1.3 (Vin), U3.4 (Vin), U5.3 (Vin)
- new net TRIG0_0: D5.1, F3.1, U8.20 (D4(PA08(I2C/AIN16/SER0:0+)))
- new net TRIG0_0_IO: F3.2, J2.1 (Pin_1)
- new net TRIG0_1: D4.1, F2.1, R4.1, U8.21 (D3(PA09(I2C/AIN17/SER0:1+)))
- new net TRIG0_1_IO: F2.2, J1.1 (Pin_1)
- new net TRIG1_0: D10.1, F8.1, U8.16 (D8(PA06/AIN6/SER0:2/TC1:0))
- new net TRIG1_0_IO: F8.2, J2.2 (Pin_2)
- new net TRIG1_1: D9.1, F7.1, R5.1, U8.15 (D9(PA07/AIN7/SER0:3/TC1:1)))
- new net TRIG1_1_IO: F7.2, J1.2 (Pin_2)
- new net TRIG4_0: D14.1, F12.1, U8.13 (A1(PB08(AIN2/SER4:0/TC4:0)))
- new net TRIG4_0_IO: F12.2, J2.3 (Pin_3)
- new net TRIG4_1: D13.1, F11.1, R6.1, U8.12 (A2(PB09(AIN3/SER4:1/TC4:1)))
- new net TRIG4_1_IO: F11.2, J1.3 (Pin_3)
- new net ~{12V_ENABLE}: U8.18 (D6(PA20(SER5:2+)))
- new net ~{5V_ENABLE}: U3.5 (EN), U5.4 (EN), U8.38 (ANT(PA13(I2C/SER2:1+)))
- new net ~{STROBE_ENABLE}: U8.17 (D7(PA21(SER5:3+)))
- no-connect marks 0 -> 14
Other:
- removed sheet LTC1760_A
- removed sheet LTC1760_B
- removed sheet sheet6090344F
- removed sheet sheet60903454
- added sheet Adafruit_BME280 (Adafruit_BME280.kicad_sch)
- added sheet Adafruit_INA260 (Adafruit_INA260_sch.kicad_sch)
- added sheet Adafruit_INA260_1 (Adafruit_INA260_sch.kicad_sch)
- added sheet BatterySystem (BatterySystem.kicad_sch)
- added sheet COMMS (COMMS.kicad_sch)
- added sheet CameraPower (CameraPower.kicad_sch)
- added sheet DS3231 (DS3231.kicad_sch)
- added sheet HighSideSwitch_LTC4412HV (HighSideSwitch_LTC4412HV.kicad_sch)
- note added: "12V Camera/Compute Power"
- note added: "5V Camera/Compute Power"
- note added: "5V MCU Power"
- note added: "BME280 Env Sensor"
- note added: "DS3231 Prrecision RTC"
- note added: "Input / Output"
- note added: "Microcontroller"
- note added: "PGND is protected for reverse polarity"
- note added: "Power Input Protection, Ideal Diodes, and Monitoring"
- note added: "SD Card"
- note added: "TTL and RS-232 COMMS"
- note removed: "Reverse Polairty Protection"
- company: Guatek -> (none)
- title: WW-Battery-Pack PCBs -> Console-Controller

Commit message: slight updates to LTC1670 modules (2 resistors added) finalizing console controller and strobe controller
Parts:
- removed D2, D3: ORG 1.8V@1mA, LED_SMD:LED_0603_1608Metric, symbol Device:LED_Small_ALT
- removed J13: STRB_PWR, Connector_Molex:Molex_Nano-Fit_105309-xx02_1x02_P2.50mm_Vertical, symbol Connector_Generic:Conn_01x02
- removed J14: CAM_COMPUTE_PWR, Connector_Molex:Molex_Nano-Fit_105309-xx02_1x02_P2.50mm_Vertical, symbol Connector_Generic:Conn_01x02
- removed J15: 5V_5A_PWR, Connector_Molex:Molex_Nano-Fit_105309-xx02_1x02_P2.50mm_Vertical, symbol Connector_Generic:Conn_01x02
- removed J16: 5V_2.5A_PWR, Connector_Molex:Molex_Nano-Fit_105309-xx02_1x02_P2.50mm_Vertical, symbol Connector_Generic:Conn_01x02
- removed J2: TRIG_IO, Connector_Molex:Molex_Nano-Fit_105310-xx06_2x03_P2.50mm_Vertical, symbol Dual-Mag-Camera-Control-rescue:Conn_01x06-SPC-Control-rescue
- removed J3: ADC_DAC, Connector_Molex:Molex_Nano-Fit_105310-xx06_2x03_P2.50mm_Vertical, symbol Dual-Mag-Camera-Control-rescue:Conn_01x06-SPC-Control-rescue
- removed J4: GPIO, Connector_Molex:Molex_Nano-Fit_105310-xx06_2x03_P2.50mm_Vertical, symbol Dual-Mag-Camera-Control-rescue:Conn_01x06-SPC-Control-rescue
- removed R2, R3: 3240, Resistor_SMD:R_0603_1608Metric_Pad1.05x0.95mm_HandSolder, symbol Device:R_Small_US
- removed U1: D24V10F5, ProjectFootprints:D24V10F5, symbol Dual-Mag-Camera-Control-rescue:D24V10F5-ProjectDevices
- removed U3: D24V50F5, ProjectFootprints:D24V50F5, symbol Dual-Mag-Camera-Control-rescue:D24V50F5-ProjectDevices
- removed U5: D24V22F5, ProjectFootprints:D24V22F5, symbol Dual-Mag-Camera-Control-rescue:D24V22F5-ProjectDevices
- added J?: DISP 12V Out, Connector_Molex:Molex_Nano-Fit_105314-xx04_2x02_P2.50mm_Horizontal, symbol Connector_Generic:Conn_02x02_Top_Bottom
- added J?: GPIO, Connector_Molex:Molex_PicoBlade_53261-0571_1x05-1MP_P1.25mm_Horizontal, symbol Dual-Mag-Camera-Control-rescue:Conn_01x06-SPC-Control-rescue
- added J?: ORIN 12V Out, Connector_Molex:Molex_Nano-Fit_105314-xx04_2x02_P2.50mm_Horizontal, symbol Connector_Generic:Conn_02x02_Top_Bottom
- added J?: ADC_DAC, Connector_Molex:Molex_PicoBlade_53261-0571_1x05-1MP_P1.25mm_Horizontal, symbol Dual-Mag-Camera-Control-rescue:Conn_01x06-SPC-Control-rescue
- added J?: COAX 12V Out, Connector_Molex:Molex_Nano-Fit_105314-xx04_2x02_P2.50mm_Horizontal, symbol Connector_Generic:Conn_02x02_Top_Bottom
- added J?: TRIG_IO_1, Connector_Molex:Molex_PicoBlade_53261-0571_1x05-1MP_P1.25mm_Horizontal, symbol Dual-Mag-Camera-Control-rescue:Conn_01x06-SPC-Control-rescue
- added J?: Probe Pwr Out, Connector_Molex:Molex_Nano-Fit_105314-xx04_2x02_P2.50mm_Horizontal, symbol Connector_Generic:Conn_02x02_Top_Bottom
- added U?: D36V28F5, ProjectFootprints:D36V28F5, symbol ProjectDevices:D36V28F5
- J1: value ~TRIG_IO -> TRIG_IO_0; footprint Connector_Molex:Molex_Nano-Fit_105310-xx06_2x03_P2.50mm_Vertical -> Connector_Molex:Molex_PicoBlade_53261-0571_1x05-1MP_P1.25mm_Horizontal; Link https://www.digikey.com/en/products/detail/molex/1053102306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 -> https://www.digikey.com/en/products/detail/molex/0532614005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; Part Number WM15076-ND -> 900-0532614005CT-ND
Connections:
- net 3.3V_LDO: now also J?.4 (Pin_4), J?.4 (Pin_4), J?.5 (Pin_5)
- net 5V_reg: now also J?.5 (Pin_5), J?.5 (Pin_5), U?.1 (Vout)
- net A3_IO: now also J?.1 (Pin_1)
- net A4_IO: now also J?.2 (Pin_2)
- net A5_IO: now also J?.3 (Pin_3)
- net DAC_OUT_IO: now also J?.4 (Pin_4)
- net GND: now also J?.3 (Pin_3), J?.4 (Pin_4), J?.6 (Pin_6), J?.6 (Pin_6), J?.6 (Pin_6), U?.2 (GND), U?.3 (GND)
- net GPIO_1_IO: now also J?.1 (Pin_1)
- net GPIO_2_IO: now also J?.2 (Pin_2)
- net GPIO_3_IO: now also J?.3 (Pin_3)
- net SystemVin: now also U?.4 (Vin), U?.5 (EN)
- net TRIG0_0_IO: now also J?.1 (Pin_1)
- net TRIG1_0_IO: now also J?.2 (Pin_2)
- net TRIG4_0_IO: now also J?.3 (Pin_3)
- net ~{STROBE_ENABLE}: no longer U8.17 (D7(PA21(SER5:3+)))
- net at D1.2 (A), R1.2: now also U?.6 (PG)
- net ~{12V_ENABLE} renamed ORIN_ENABLE
- net ~{5V_ENABLE} renamed CAM_ENABLE
- new net DC-Reg-i7C-12V/PGND_Out: J?.3 (Pin_3), J?.4 (Pin_4)
- new net DC-Reg-i7C-12V/Vout: J?.1 (Pin_1), J?.2 (Pin_2)
- new net DC-Reg-i7C-12V1/PGND_Out: J?.3 (Pin_3), J?.4 (Pin_4)
- new net DC-Reg-i7C-12V1/Vout: J?.1 (Pin_1), J?.2 (Pin_2)
- new net DC-Reg-i7C-12V2/PGND_Out: J?.3 (Pin_3), J?.4 (Pin_4)
- new net DC-Reg-i7C-12V2/Vout: J?.1 (Pin_1), J?.2 (Pin_2)
- new net DISP_ENABLE: U8.17 (D7(PA21(SER5:3+)))
- new net ProbeVout: J?.1 (Pin_1), J?.2 (Pin_2)
- no-connect marks 14 -> 12
Other:
- removed sheet CameraPower
- added sheet DC-Reg-i7C-12V (DC-Reg-i7C-12V.kicad_sch)
- added sheet DC-Reg-i7C-12V1 (DC-Reg-i7C-12V.kicad_sch)
- added sheet DC-Reg-i7C-12V2 (DC-Reg-i7C-12V.kicad_sch)
- sheet COMMS ports: added 3V3; removed 3.3V
- note removed: "5V Camera/Compute Power"
- moved on the sheet: D1, R1, U4
