File: LTC1760-Module/LTC1760-Module.kicad_sch (KiCad schematic)
At the start: 73 parts, among them J1 Battery 1, J2 Battery 1, J3 Parallel-I/O, J4 System-I/O, J5 Power-I/O, Q1 Si7141DP, Q2 Si7141DP, U1 FDS6990, U2 FDS6990, U3 FDS4935BZ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

Commit message: slight updates to LTC1670 modules (2 resistors added) finalizing console controller and strobe controller
Parts:
- added R? (x2): 280k 1%, Resistor_SMD:R_0603_1608Metric, symbol Device:R_Small_US
Connections:
- net ~{BAT_EN1}: now also R?.2; no longer Q1.4 (G), R15.2
- net ~{BAT_EN2}: now also R?.2; no longer Q2.4 (G), R16.2
- new net: Q2.4 (G), R16.2, R?.1
- new net: Q1.4 (G), R15.2, R?.1
Other:
- title: (none) -> LTC1760 Module
Changed lines of the file:
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@@
 (kicad_sch (version 20211123) (generator eeschema)
   (paper "A4")
+  (title_block
+    (title "LTC1760 Module")
+    (date "2023-02-05")
+    (rev "A")
+  )
   (junction (at 149.86 172.72) (diameter 0) (color 0 0 0 0)
   )
@@
   (junction (at 50.8 149.86) (diameter 0) (color 0 0 0 0)
   )
-  (junction (at 96.52 167.64) (diameter 0) (color 0 0 0 0)
-  )
   (junction (at 104.14 182.88) (diameter 0) (color 0 0 0 0)
   )
@@
   (junction (at 78.74 41.91) (diameter 0) (color 0 0 0 0)
   )
+  (junction (at 96.52 167.64) (diameter 0) (color 0 0 0 0)
+  )
   (junction (at 38.1 138.43) (diameter 0) (color 0 0 0 0)
   )
@@
     (stroke (width 0) (type default) (color 0 0 0 0))
   )
+  (wire (pts (xy 93.98 167.64) (xy 96.52 167.64))
+    (stroke (width 0) (type default) (color 0 0 0 0))
+  )
   (wire (pts (xy 72.39 62.23) (xy 76.2 62.23))
     (stroke (width 0) (type default) (color 0 0 0 0))
@@
     (stroke (width 0) (type default) (color 0 0 0 0))
   )
-  (wire (pts (xy 96.52 128.27) (xy 91.44 128.27))
+  (wire (pts (xy 96.52 128.27) (xy 93.98 128.27))
     (stroke (width 0) (type default) (color 0 0 0 0))
   )
@@
     (stroke (width 0) (type default) (color 0 0 0 0))
   )
+  (wire (pts (xy 86.36 128.27) (xy 88.9 128.27))
+    (stroke (width 0) (type default) (color 0 0 0 0))
+  )
   (wire (pts (xy 251.46 138.43) (xy 264.16 138.43))
     (stroke (width 0) (type default) (color 0 0 0 0))
@@
     (stroke (width 0) (type default) (color 0 0 0 0))
   )
-  (wire (pts (xy 96.52 167.64) (xy 91.44 167.64))
-    (stroke (width 0) (type default) (color 0 0 0 0))
-  )
   (wire (pts (xy 120.65 39.37) (xy 118.11 39.37))
     (stroke (width 0) (type default) (color 0 0 0 0))
@@
     (stroke (width 0) (type default) (color 0 0 0 0))
   )
+  (wire (pts (xy 86.36 167.64) (xy 88.9 167.64))
+    (stroke (width 0) (type default) (color 0 0 0 0))
+  )
   (wire (pts (xy 50.8 149.86) (xy 50.8 142.24))
     (stroke (width 0) (type default) (color 0 0 0 0))
@@
     (effects (font (size 1.27 1.27)) (justify right))
   )
-  (hierarchical_label "~{BAT_EN2}" (shape input) (at 91.44 167.64 180)
+  (hierarchical_label "~{BAT_EN2}" (shape input) (at 86.36 167.64 180)
     (effects (font (size 1.27 1.27)) (justify right))
   )
@@
     (effects (font (size 1.27 1.27)) (justify right))
   )
-  (hierarchical_label "~{BAT_EN1}" (shape input) (at 91.44 128.27 180)
+  (hierarchical_label "~{BAT_EN1}" (shape input) (at 86.36 128.27 180)
     (effects (font (size 1.27 1.27)) (justify right))
   )
@@
     (pin "1")
   )
+  (symbol (lib_id "Device:R_Small_US") (at 91.44 128.27 270) (unit 1)
+    (in_bom yes) (on_board yes)
+    (property "Reference" "R?" (id 0) (at 90.17 123.19 90)
+      (effects (font (size 1.27 1.27)) (justify left))
+    )
+    (property "Value" "280k 1%" (id 1) (at 87.63 125.73 90)
+      (effects (font (size 1.27 1.27)) (justify left))
+    )
+    (property "Footprint" "Resistor_SMD:R_0603_1608Metric" (id 2) (at 91.44 128.27 0)
+      (effects (font (size 1.27 1.27)) hide)
+    )
+    (property "Datasheet" "https://industrial.panasonic.com/cdbs/www-data/pdf/RDA0000/AOA0000C304.pdf" (id 3) (at 91.44 128.27 0)
+      (effects (font (size 1.27 1.27)) hide)
+    )
+    (property "Part Number" "P280KHCT-ND" (id 4) (at 91.44 128.27 0)
+      (effects (font (size 1.27 1.27)) hide)
+    )
+    (property "Supplier" "Digikey" (id 5) (at 91.44 128.27 0)
+      (effects (font (size 1.27 1.27)) hide)
+    )
+    (property "Link" "https://www.digikey.com/product-detail/en/panasonic-electronic-components/ERJ-3EKF2803V/P280KHCT-ND/198299" (id 6) (at 91.44 128.27 0)
+      (effects (font (size 1.27 1.27)) hide)
+    )
+    (pin "1")
+    (pin "2")
+  )
   (symbol (lib_id "Mechanical:MountingHole_Pad") (at 153.67 193.04 0) (unit 1)
     (in_bom yes) (on_board yes) (fields_autoplaced)
@@
     (pin "1")
   )
+  (symbol (lib_id "Device:R_Small_US") (at 91.44 167.64 270) (unit 1)
+    (in_bom yes) (on_board yes)
+    (property "Reference" "R?" (id 0) (at 90.17 162.56 90)
+      (effects (font (size 1.27 1.27)) (justify left))
+    )
+    (property "Value" "280k 1%" (id 1) (at 87.63 165.1 90)
+      (effects (font (size 1.27 1.27)) (justify left))
+    )
+    (property "Footprint" "Resistor_SMD:R_0603_1608Metric" (id 2) (at 91.44 167.64 0)
+      (effects (font (size 1.27 1.27)) hide)
+    )
+    (property "Datasheet" "https://industrial.panasonic.com/cdbs/www-data/pdf/RDA0000/AOA0000C304.pdf" (id 3) (at 91.44 167.64 0)
+      (effects (font (size 1.27 1.27)) hide)
+    )
+    (property "Part Number" "P280KHCT-ND" (id 4) (at 91.44 167.64 0)
+      (effects (font (size 1.27 1.27)) hide)
+    )
+    (property "Supplier" "Digikey" (id 5) (at 91.44 167.64 0)
+      (effects (font (size 1.27 1.27)) hide)
+    )
+    (property "Link" "https://www.digikey.com/product-detail/en/panasonic-electronic-components/ERJ-3EKF2803V/P280KHCT-ND/198299" (id 6) (at 91.44 167.64 0)
+      (effects (font (size 1.27 1.27)) hide)
+    )
+    (pin "1")
+    (pin "2")
+  )
   (sheet (at 242.57 22.86) (size 12.7 8.89) (fields_autoplaced)
     (stroke (width 0) (type solid) (color 0 0 0 0))
@@
       (reference "Q2") (unit 1) (value "Si7141DP") (footprint "Package_SO:PowerPAK_SO-8_Single")
     )
-    (path "/b7eb4f8f-cb1f-46c5-a151-471baa53c09b/00000000-0000-0000-0000-00005ec89eff"
-      (reference "Q3") (unit 1) (value "Si7463DP") (footprint "Package_SO:PowerPAK_SO-8_Single")
+    (path "/b7eb4f8f-cb1f-46c5-a151-471baa53c09b/328805fd-9276-42ac-96e7-ed961a2645ce"
+      (reference "Q?") (unit 1) (value "Si7141DP") (footprint "Package_SO:PowerPAK_SO-8_Single")
     )
     (path "/00000000-0000-0000-0000-00005f733b8d"
@@
       (reference "R26") (unit 1) (value "470k") (footprint "Resistor_SMD:R_0603_1608Metric_Pad1.05x0.95mm_HandSolder")
     )
+    (path "/cd2d2fb2-9aca-41f0-be21-42fed54a3cf3"
+      (reference "R?") (unit 1) (value "280k 1%") (footprint "Resistor_SMD:R_0603_1608Metric")
+    )
+    (path "/f487808c-3e4e-41c4-a1f4-b02337ae2310"
+      (reference "R?") (unit 1) (value "280k 1%") (footprint "Resistor_SMD:R_0603_1608Metric")
+    )
     (path "/00000000-0000-0000-0000-00005eebdde0"
